File: KiCad9/DAC8734/power_supply.kicad_sch (KiCad schematic)
At the start: 5 parts, among them U6 TPS62745DSSR

Commit message: spice
Parts:
- U6: DIGIKEY PN 490-10639-1-ND -> 296-44339-1-ND
Changed lines of the file:
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@@
 			)
 		)
-		(property "DIGIKEY PN" "490-10639-1-ND"
+		(property "DIGIKEY PN" "296-44339-1-ND"
 			(at 163.83 80.01 0)
 			(effects
